File: attiny85_4Transistor.sch (EAGLE design)
At the start: 27 parts, among them Q1 BC817-16SMD, Q3 BC817-16SMD, Q4 BC817-16SMD, Q5 BC817-16SMD, U2 Tiny45-20-SMT, U3 V_REG_317SMD

Commit message: add programing
Parts:
- PC1, PC2: value 47u -> 27u
- R1, R3, R5, R8: value (none) -> 1K
- R10, R6, R7, R9: value (none) -> 10K
Changed lines of the file:
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@@
 <part name="C2" library="SparkFun-Capacitors" deviceset="1.0UF-25V-+80/-20(0805)" device="" value="1.0uF"/>
 <part name="GND7" library="supply1" deviceset="GND" device=""/>
-<part name="PC1" library="rcl" deviceset="CPOL-EU" device="E2.5-5V" value="47u"/>
+<part name="PC1" library="rcl" deviceset="CPOL-EU" device="E2.5-5V" value="27u"/>
 <part name="GND9" library="supply1" deviceset="GND" device=""/>
 <part name="GND11" library="supply1" deviceset="GND" device=""/>
 <part name="P+8" library="supply1" deviceset="+5V" device=""/>
 <part name="P+1" library="supply1" deviceset="+5V" device=""/>
-<part name="PC2" library="rcl" deviceset="CPOL-EU" device="E2.5-5V" value="47u"/>
+<part name="PC2" library="rcl" deviceset="CPOL-EU" device="E2.5-5V" value="27u"/>
 <part name="Q1" library="transistor-npn" deviceset="BC817*" device="SMD" technology="-16"/>
 <part name="Q3" library="transistor-npn" deviceset="BC817*" device="SMD" technology="-16"/>
-<part name="R1" library="rcl" deviceset="R-US_" device="R0805"/>
-<part name="R3" library="rcl" deviceset="R-US_" device="R0805"/>
-<part name="R7" library="adafruit" deviceset="R-US_" device="M0805"/>
-<part name="R9" library="adafruit" deviceset="R-US_" device="M0805"/>
+<part name="R1" library="rcl" deviceset="R-US_" device="R0805" value="1K"/>
+<part name="R3" library="rcl" deviceset="R-US_" device="R0805" value="1K"/>
+<part name="R7" library="adafruit" deviceset="R-US_" device="M0805" value="10K"/>
+<part name="R9" library="adafruit" deviceset="R-US_" device="M0805" value="10K"/>
 <part name="GND1" library="supply1" deviceset="GND" device=""/>
 <part name="GND2" library="supply1" deviceset="GND" device=""/>
@@
 <part name="GND5" library="supply1" deviceset="GND" device=""/>
 <part name="Q4" library="transistor-npn" deviceset="BC817*" device="SMD" technology="-16"/>
-<part name="R5" library="rcl" deviceset="R-US_" device="R0805"/>
-<part name="R6" library="adafruit" deviceset="R-US_" device="M0805"/>
+<part name="R5" library="rcl" deviceset="R-US_" device="R0805" value="1K"/>
+<part name="R6" library="adafruit" deviceset="R-US_" device="M0805" value="10K"/>
 <part name="GND6" library="supply1" deviceset="GND" device=""/>
 <part name="Q5" library="transistor-npn" deviceset="BC817*" device="SMD" technology="-16"/>
-<part name="R8" library="rcl" deviceset="R-US_" device="R0805"/>
-<part name="R10" library="adafruit" deviceset="R-US_" device="M0805"/>
+<part name="R8" library="rcl" deviceset="R-US_" device="R0805" value="1K"/>
+<part name="R10" library="adafruit" deviceset="R-US_" device="M0805" value="10K"/>
 <part name="GND8" library="supply1" deviceset="GND" device=""/>
 <part name="PAD1" library="wirepad" deviceset="2,15/1,0" device=""/>
